Commit message: update Franka Panda URDF with merged/simplified/textured meshes. Each of the 11 links have their own single OBJ mesh (8 links + hand + 2 fingers)

File: omniisaacgymenvs/franka_panda.urdf (robot description, URDF)
Before this commit: robot panda, 12 links, 11 joints
Links:
- link hand: geometry collision mesh filename=franka_description/meshes/collision/hand.obj; visual mesh filename=franka_description/meshes/visual/hand_new.obj
- link leftfinger: geometry collision mesh filename=franka_description/meshes/collision/finger.obj; visual mesh filename=franka_description/meshes/visual/finger_new.obj
- link panda_link0: geometry collision mesh filename=franka_description/meshes/collision/link0.obj; visual mesh filename=franka_description/meshes/visual/link0_new.obj
- link panda_link1: geometry collision mesh filename=franka_description/meshes/collision/link1.obj; visual mesh filename=franka_description/meshes/visual/link1_new.obj
- link panda_link2: geometry collision mesh filename=franka_description/meshes/collision/link2.obj; visual mesh filename=franka_description/meshes/visual/link2_new.obj
- link panda_link3: geometry collision mesh filename=franka_description/meshes/collision/link3.obj; visual mesh filename=franka_description/meshes/visual/link3_new.obj
- link panda_link4: geometry collision mesh filename=franka_description/meshes/collision/link4.obj; visual mesh filename=franka_description/meshes/visual/link4_new.obj
- link panda_link5: geometry collision mesh filename=franka_description/meshes/collision/link5.obj; visual mesh filename=franka_description/meshes/visual/link5_new.obj
- link panda_link6: geometry collision mesh filename=franka_description/meshes/collision/link6.obj; visual mesh filename=franka_description/meshes/visual/link6_new.obj
- link panda_link7: geometry collision mesh filename=franka_description/meshes/collision/link7.obj; visual mesh filename=franka_description/meshes/visual/link7_new.obj
- link rightfinger: geometry collision mesh filename=franka_description/meshes/collision/finger.obj; visual mesh filename=franka_description/meshes/visual/finger_new.obj
